Commit message: feat: add soarm_control package; fix so101 joint names; drop vel/accel interfaces
soarm_control (new package):
- CMakeLists.txt and package.xml
- config/so100_controllers.yaml: ForwardCommandController for 6 joints
  (shoulder_pan_joint, shoulder_lift_joint, elbow_flex_joint, wrist_flex_joint,
  wrist_roll_joint, gripper_joint) with position interface
- config/so101_controllers.yaml: same joint names (now with _joint suffix)
- launch/soarm.launch.py: model arg (so100/so101, default: so101) selects
  URDF and controller config dynamically; use_mock defaults to true;
  starts RSP, controller_manager, joint_state_broadcaster, soarm_controller,
  and motor diagnostics (TimerAction-staggered)

soarm_description:
- so101.urdf.xacro: rename 5 revolute joints (shoulder_pan, shoulder_lift,
  elbow_flex, wrist_flex, wrist_roll, gripper) to *_joint suffix to match
  so100 naming convention; applies to both URDF joints and ros2_control joints
- so100.urdf.xacro + so101.urdf.xacro: remove velocity and acceleration
  command interfaces — only position is needed (ForwardCommandController
  only claims position; STS vel/accel params not used by any standard
  ros2_control controller)

File: soarm_description/urdf/so100/so100.urdf.xacro (robot description, xacro)
@@ -253,6 +253,4 @@
       <param name="position_center_steps">2048</param>
       <command_interface name="position"/>
-      <command_interface name="velocity"/>
-      <command_interface name="acceleration"/>
       <state_interface name="position"/>
       <state_interface name="velocity"/>
@@ -271,6 +269,4 @@
       <param name="position_center_steps">2048</param>
       <command_interface name="position"/>
-      <command_interface name="velocity"/>
-      <command_interface name="acceleration"/>
       <state_interface name="position"/>
       <state_interface name="velocity"/>
@@ -289,6 +285,4 @@
       <param name="position_center_steps">2048</param>
       <command_interface name="position"/>
-      <command_interface name="velocity"/>
-      <command_interface name="acceleration"/>
       <state_interface name="position"/>
       <state_interface name="velocity"/>
@@ -307,6 +301,4 @@
       <param name="position_center_steps">2048</param>
       <command_interface name="position"/>
-      <command_interface name="velocity"/>
-      <command_interface name="acceleration"/>
       <state_interface name="position"/>
       <state_interface name="velocity"/>
@@ -325,6 +317,4 @@
       <param name="position_center_steps">2048</param>
       <command_interface name="position"/>
-      <command_interface name="velocity"/>
-      <command_interface name="acceleration"/>
       <state_interface name="position"/>
       <state_interface name="velocity"/>
@@ -343,6 +333,4 @@
       <param name="position_center_steps">2048</param>
       <command_interface name="position"/>
-      <command_interface name="velocity"/>
-      <command_interface name="acceleration"/>
       <state_interface name="position"/>
       <state_interface name="velocity"/>

File: soarm_description/urdf/so101/so101.urdf.xacro (robot description, xacro)
@@ -300,5 +300,5 @@
   </link>
   <!-- JOINTS -->
-  <joint name="shoulder_pan" type="revolute">
+  <joint name="shoulder_pan_joint" type="revolute">
     <parent link="base_link"/>
     <child link="shoulder_link"/>
@@ -307,5 +307,5 @@
     <limit lower="${shoulder_pan_lower}" upper="${shoulder_pan_upper}" effort="${max_torque_nm}" velocity="${max_velocity_rads}"/>
   </joint>
-  <joint name="shoulder_lift" type="revolute">
+  <joint name="shoulder_lift_joint" type="revolute">
     <parent link="shoulder_link"/>
     <child link="upper_arm_link"/>
@@ -314,5 +314,5 @@
     <limit lower="${shoulder_lift_lower}" upper="${shoulder_lift_upper}" effort="${max_torque_nm}" velocity="${max_velocity_rads}"/>
   </joint>
-  <joint name="elbow_flex" type="revolute">
+  <joint name="elbow_flex_joint" type="revolute">
     <parent link="upper_arm_link"/>
     <child link="lower_arm_link"/>
@@ -321,5 +321,5 @@
     <limit lower="${elbow_flex_lower}" upper="${elbow_flex_upper}" effort="${max_torque_nm}" velocity="${max_velocity_rads}"/>
   </joint>
-  <joint name="wrist_flex" type="revolute">
+  <joint name="wrist_flex_joint" type="revolute">
     <parent link="lower_arm_link"/>
     <child link="wrist_link"/>
@@ -328,5 +328,5 @@
     <limit lower="${wrist_flex_lower}" upper="${wrist_flex_upper}" effort="${max_torque_nm}" velocity="${max_velocity_rads}"/>
   </joint>
-  <joint name="wrist_roll" type="revolute">
+  <joint name="wrist_roll_joint" type="revolute">
     <parent link="wrist_link"/>
     <child link="gripper_link"/>
@@ -340,5 +340,5 @@
     <origin xyz="${gripper_frame_xyz}" rpy="${gripper_frame_rpy}"/>
   </joint>
-  <joint name="gripper" type="revolute">
+  <joint name="gripper_joint" type="revolute">
     <parent link="gripper_link"/>
     <child link="moving_jaw_link"/>
@@ -359,5 +359,5 @@
       <param name="reset_states_on_activate">true</param>
     </hardware>
-    <joint name="shoulder_pan">
+    <joint name="shoulder_pan_joint">
       <param name="motor_id">${shoulder_pan_motor_id}</param>
       <param name="operating_mode">${operating_mode}</param>
@@ -367,15 +367,13 @@
       <param name="position_center_steps">2048</param>
       <command_interface name="position"/>
-      <command_interface name="velocity"/>
-      <command_interface name="acceleration"/>
-      <state_interface name="position"/>
-      <state_interface name="velocity"/>
-      <state_interface name="effort"/>
-      <state_interface name="voltage"/>
-      <state_interface name="temperature"/>
-      <state_interface name="current"/>
-      <state_interface name="is_moving"/>
-    </joint>
-    <joint name="shoulder_lift">
+      <state_interface name="position"/>
+      <state_interface name="velocity"/>
+      <state_interface name="effort"/>
+      <state_interface name="voltage"/>
+      <state_interface name="temperature"/>
+      <state_interface name="current"/>
+      <state_interface name="is_moving"/>
+    </joint>
+    <joint name="shoulder_lift_joint">
       <param name="motor_id">${shoulder_lift_motor_id}</param>
       <param name="operating_mode">${operating_mode}</param>
@@ -385,15 +383,13 @@
       <param name="position_center_steps">2048</param>
       <command_interface name="position"/>
-      <command_interface name="velocity"/>
-      <command_interface name="acceleration"/>
-      <state_interface name="position"/>
-      <state_interface name="velocity"/>
-      <state_interface name="effort"/>
-      <state_interface name="voltage"/>
-      <state_interface name="temperature"/>
-      <state_interface name="current"/>
-      <state_interface name="is_moving"/>
-    </joint>
-    <joint name="elbow_flex">
+      <state_interface name="position"/>
+      <state_interface name="velocity"/>
+      <state_interface name="effort"/>
+      <state_interface name="voltage"/>
+      <state_interface name="temperature"/>
+      <state_interface name="current"/>
+      <state_interface name="is_moving"/>
+    </joint>
+    <joint name="elbow_flex_joint">
       <param name="motor_id">${elbow_flex_motor_id}</param>
       <param name="operating_mode">${operating_mode}</param>
@@ -403,15 +399,13 @@
       <param name="position_center_steps">2048</param>
       <command_interface name="position"/>
-      <command_interface name="velocity"/>
-      <command_interface name="acceleration"/>
-      <state_interface name="position"/>
-      <state_interface name="velocity"/>
-      <state_interface name="effort"/>
-      <state_interface name="voltage"/>
-      <state_interface name="temperature"/>
-      <state_interface name="current"/>
-      <state_interface name="is_moving"/>
-    </joint>
-    <joint name="wrist_flex">
+      <state_interface name="position"/>
+      <state_interface name="velocity"/>
+      <state_interface name="effort"/>
+      <state_interface name="voltage"/>
+      <state_interface name="temperature"/>
+      <state_interface name="current"/>
+      <state_interface name="is_moving"/>
+    </joint>
+    <joint name="wrist_flex_joint">
       <param name="motor_id">${wrist_flex_motor_id}</param>
       <param name="operating_mode">${operating_mode}</param>
@@ -421,15 +415,13 @@
       <param name="position_center_steps">2048</param>
       <command_interface name="position"/>
-      <command_interface name="velocity"/>
-      <command_interface name="acceleration"/>
-      <state_interface name="position"/>
-      <state_interface name="velocity"/>
-      <state_interface name="effort"/>
-      <state_interface name="voltage"/>
-      <state_interface name="temperature"/>
-      <state_interface name="current"/>
-      <state_interface name="is_moving"/>
-    </joint>
-    <joint name="wrist_roll">
+      <state_interface name="position"/>
+      <state_interface name="velocity"/>
+      <state_interface name="effort"/>
+      <state_interface name="voltage"/>
+      <state_interface name="temperature"/>
+      <state_interface name="current"/>
+      <state_interface name="is_moving"/>
+    </joint>
+    <joint name="wrist_roll_joint">
       <param name="motor_id">${wrist_roll_motor_id}</param>
       <param name="operating_mode">${operating_mode}</param>
@@ -439,15 +431,13 @@
       <param name="position_center_steps">2048</param>
       <command_interface name="position"/>
-      <command_interface name="velocity"/>
-      <command_interface name="acceleration"/>
-      <state_interface name="position"/>
-      <state_interface name="velocity"/>
-      <state_interface name="effort"/>
-      <state_interface name="voltage"/>
-      <state_interface name="temperature"/>
-      <state_interface name="current"/>
-      <state_interface name="is_moving"/>
-    </joint>
-    <joint name="gripper">
+      <state_interface name="position"/>
+      <state_interface name="velocity"/>
+      <state_interface name="effort"/>
+      <state_interface name="voltage"/>
+      <state_interface name="temperature"/>
+      <state_interface name="current"/>
+      <state_interface name="is_moving"/>
+    </joint>
+    <joint name="gripper_joint">
       <param name="motor_id">${gripper_motor_id}</param>
       <param name="operating_mode">${operating_mode}</param>
@@ -457,6 +447,4 @@
       <param name="position_center_steps">2048</param>
       <command_interface name="position"/>
-      <command_interface name="velocity"/>
-      <command_interface name="acceleration"/>
       <state_interface name="position"/>
       <state_interface name="velocity"/>
