Commit message: Add base_footprint root link to so100 and so101 URDFs

File: soarm_description/urdf/so100/so100.urdf (robot description, URDF)
Before this commit: robot so100, 7 links, 6 joints
Links:
- added link base_footprint
Joints:
- added joint base_footprint_joint: type fixed, parent base_footprint, child base_link, origin xyz=0 0 0 rpy=0 0 0

File: soarm_description/urdf/so100/so100.urdf.xacro (robot description, xacro)
@@ -14,4 +14,11 @@
   </material>
   <!-- LINKS -->
+  <!-- Dummy root link (KDL does not support inertia on root link) -->
+  <link name="base_footprint"/>
+  <joint name="world_to_base" type="fixed">
+    <parent link="base_footprint"/>
+    <child link="base_link"/>
+    <origin xyz="0 0 0" rpy="0 0 0"/>
+  </joint>
   <!-- Base link -->
   <link name="base_link">

File: soarm_description/urdf/so101/so101.urdf (robot description, URDF)
Before this commit: robot so101, 8 links, 7 joints
Links:
- added link base_footprint
Joints:
- added joint base_footprint_joint: type fixed, parent base_footprint, child base_link, origin xyz=0 0 0 rpy=0 0 0

File: soarm_description/urdf/so101/so101.urdf.xacro (robot description, xacro)
@@ -14,4 +14,11 @@
   </material>
   <!-- LINKS -->
+  <!-- Dummy root link (KDL does not support inertia on root link) -->
+  <link name="base_footprint"/>
+  <joint name="world_to_base" type="fixed">
+    <parent link="base_footprint"/>
+    <child link="base_link"/>
+    <origin xyz="0 0 0" rpy="0 0 0"/>
+  </joint>
   <!-- Base link -->
   <link name="base_link">
