Commit message: Fold so_arm_shared.xml into so_arm.mjcf.xacro and trim verbose comments

File: so_arm_description/mjcf/so_arm.mjcf.xacro (robot description, xacro)
@@ -1,17 +1,39 @@
 <?xml version="1.0"?>
-<!-- Parametric SO-100/SO-101 MJCF assembly (mujoco_ros2_control equivalent of so100/so101
-     urdf.xacro): so_arm100_body/so_arm101_body macros, selected by so_arm_config; standalone
-     mode (default) wraps the selected one in worldbody + floor/lighting.
-     Body positions/inertials come from our own URDF sources, not ros2_so_arm's or MuJoCo
-     Menagerie's MJCF - those use a different joint-axis convention (plus an extra SO-101
-     gripper-pitch offset) that would desync real-hardware and sim position commands.
-     Joint dynamics/actuators live in so_arm_shared.xml (variant-independent). Usage:
-     xacro so_arm.mjcf.xacro so_arm_config:=so101 > /tmp/so_arm.xml -->
+<!-- Parametric SO-100/SO-101 MJCF assembly (mujoco_ros2_control equivalent of so100/so101 urdf.xacro).
+     Body geometry comes from our own URDF, not ros2_so_arm/MuJoCo Menagerie (different joint-axis convention).
+     Usage: xacro so_arm.mjcf.xacro so_arm_config:=so101 > /tmp/so_arm.xml -->
 <mujoco xmlns:xacro="http://www.ros.org/wiki/xacro" model="so_arm">
   <xacro:arg name="so_arm_config" default="so101"/>
   <xacro:arg name="standalone" default="true"/>
+  <!-- so101 only; mirrors urdf's wrist_camera_urdf arg. False omits the camera bodies below. -->
+  <xacro:arg name="wrist_camera_mjcf" default="true"/>
   <xacro:property name="so_arm_config" value="$(arg so_arm_config)"/>
-  <!-- xacro:include, not a plain <include> - so_arm_shared.xml is variant-independent. -->
-  <xacro:include filename="$(find so_arm_description)/mjcf/so_arm_shared.xml"/>
+  <compiler angle="radian"/>
+  <option cone="elliptic" impratio="10"/>
+  <asset>
+    <material name="light_grey" rgba="0.8 0.8 0.8 1.0"/>
+    <material name="charcoal" rgba="0.15 0.15 0.15 1.0"/>
+    <material name="transparent" rgba="1 0 0 0.3"/>
+  </asset>
+  <default>
+    <default class="sts3215">
+      <joint damping="0.60" frictionloss="0.052" armature="0.028"/>
+      <position kp="17.8" kv="0.0" forcerange="-3.35 3.35"/>
+      <default class="visual">
+        <geom type="mesh" contype="0" conaffinity="0" density="0" group="2"/>
+      </default>
+      <default class="collision">
+        <geom type="mesh" group="3" material="transparent"/>
+      </default>
+    </default>
+  </default>
+  <actuator>
+    <position class="sts3215" name="shoulder_pan_joint" joint="shoulder_pan_joint" inheritrange="1"/>
+    <position class="sts3215" name="shoulder_lift_joint" joint="shoulder_lift_joint" inheritrange="1"/>
+    <position class="sts3215" name="elbow_flex_joint" joint="elbow_flex_joint" inheritrange="1"/>
+    <position class="sts3215" name="wrist_flex_joint" joint="wrist_flex_joint" inheritrange="1"/>
+    <position class="sts3215" name="wrist_roll_joint" joint="wrist_roll_joint" inheritrange="1"/>
+    <position class="sts3215" name="gripper_joint" joint="gripper_joint" inheritrange="1"/>
+  </actuator>
   <xacro:if value="${so_arm_config == 'so100'}">
     <asset>
@@ -30,7 +52,5 @@
       <mesh name="Moving_Jaw" file="$(find so_arm_description)/meshes/so100/Moving_Jaw.stl"/>
     </asset>
-    <!-- Values verbatim from so100's URDF - joints rotate about local Z ("all-Z" convention),
-         with the child body's pos/quat compensating so meshes land where a naturally-oriented
-         joint axis would. -->
+    <!-- Values verbatim from so100's URDF; joints rotate about local Z, child pos/quat compensates. -->
     <xacro:macro name="so_arm100_body">
       <body name="base_link">
@@ -71,10 +91,8 @@
                   <inertial pos="0.00552377 -0.000483583 -0.0280167" mass="0.0929859"
                             diaginertia="5.03136e-05 2.72961e-05 4.64098e-05"/>
-                  <!-- No collision geom here or on moving_jaw_link (avoids contact-solver
-                       jitter) - unlike URDF/FCL, which covers both jaws. -->
+                  <!-- No collision geom here or on moving_jaw_link (avoids contact-solver jitter). -->
                   <geom mesh="Fixed_Jaw" material="light_grey" class="visual" quat="0.707107 0.707107 0 0"/>
                   <geom mesh="Fixed_Jaw_Motor" material="charcoal" class="visual" quat="0.707107 0.707107 0 0"/>
-                  <!-- TCP marker, matches URDF's fixed end_effector_joint (end_effector_xyz/rpy
-                       in so100.common.xacro) - estimated from Fixed_Jaw.stl, not calibrated. -->
+                  <!-- TCP marker, matches URDF's end_effector_joint; estimated, not calibrated. -->
                   <site group="5" name="end_effector_link" pos="0.0025 0.0 -0.106" quat="0.707107 0 0.707107 0"/>
                   <body name="moving_jaw_link" pos="-0.0202 0 -0.0244" quat="0 0 0.707107 0.707107">
@@ -123,6 +141,5 @@
       <mesh name="moving_jaw_so101_v1" file="$(find so_arm_description)/meshes/so101/moving_jaw_so101_v1.stl"/>
     </asset>
-    <!-- Ported from ros2_so_arm's so_arm101.xml (verified to match our own URDF for every
-         joint except gripper_joint, recomputed below from gripper_rpy - see file header). -->
+    <!-- Ported from ros2_so_arm's so_arm101.xml, verified against our URDF (gripper_joint recomputed below). -->
     <xacro:macro name="so_arm101_body">
       <body name="base_link">
@@ -193,5 +210,6 @@
                 <geom class="collision" pos="0 -0.028 0.0181" quat="0.5 -0.5 -0.5 -0.5"
                       mesh="wrist_roll_pitch_so101_v2" material="light_grey"/>
-                <body name="gripper_link" pos="0 -0.0611 0.0181" quat="0 0 0.707107 0.707107">
+                <!-- quat carries so101_new_calib.xml's wrist_roll calibration offset (matches URDF). -->
+                <body name="gripper_link" pos="0 -0.0611 0.0181" quat="0.0172091 -0.0172091 0.706897 0.706897">
                   <joint axis="0 0 1" name="wrist_roll_joint" range="-2.74385 2.84121" class="sts3215"/>
                   <inertial pos="0.000213627 0.000245138 -0.025187" mass="0.087"
@@ -205,23 +223,23 @@
                   <geom class="collision" pos="0 -0.000218214 0.000949706" quat="0 1 0 0"
                         mesh="wrist_roll_follower_so101_v1" material="light_grey"/>
-                  <body name="wrist_camera_mount_link" pos="-0.0150 0.0240 -0.0315" quat="0.499798 -0.5002 0.499802 -0.5002">
-                    <inertial pos="0 0 0" mass="0.02" diaginertia="1e-5 1e-5 1e-5"/>
-                    <geom class="visual" pos="0 0 0" quat="1 0 0 0"
-                      mesh="wrist_camera_mount_so101_v1" material="light_grey"/>
-                    <geom class="collision" pos="0 0 0" quat="1 0 0 0"
-                      mesh="wrist_camera_mount_so101_v1" material="light_grey"/>
-                    <body name="wrist_camera_body_link" pos="-0.04941 -0.03813 0.0175" quat="0.379787 -0.596458 -0.379788 -0.596456">
-                      <inertial pos="0 0 0" mass="0.015" diaginertia="1e-5 1e-5 1e-5"/>
+                  <xacro:if value="${'$(arg wrist_camera_mjcf)' == 'true'}">
+                    <body name="wrist_camera_mount_link" pos="-0.0150 0.0240 -0.0315" quat="0.499798 -0.5002 0.499802 -0.5002">
+                      <inertial pos="0 0 0" mass="0.02" diaginertia="1e-5 1e-5 1e-5"/>
                       <geom class="visual" pos="0 0 0" quat="1 0 0 0"
-                        mesh="wrist_camera_so101_v1" material="charcoal"/>
+                        mesh="wrist_camera_mount_so101_v1" material="light_grey"/>
                       <geom class="collision" pos="0 0 0" quat="1 0 0 0"
-                        mesh="wrist_camera_so101_v1" material="charcoal"/>
+                        mesh="wrist_camera_mount_so101_v1" material="light_grey"/>
+                      <body name="wrist_camera_body_link" pos="-0.04941 -0.03813 0.0175" quat="0.379787 -0.596458 -0.379788 -0.596456">
+                        <inertial pos="0 0 0" mass="0.015" diaginertia="1e-5 1e-5 1e-5"/>
+                        <geom class="visual" pos="0 0 0" quat="1 0 0 0"
+                          mesh="wrist_camera_so101_v1" material="charcoal"/>
+                        <geom class="collision" pos="0 0 0" quat="1 0 0 0"
+                          mesh="wrist_camera_so101_v1" material="charcoal"/>
+                      </body>
                     </body>
-                  </body>
-                  <!-- Matches URDF's end_effector_joint rpy, not ros2_so_arm's MJCF site (which
-                       doesn't match it). -->
+                  </xacro:if>
+                  <!-- Matches URDF's end_effector_joint rpy, unlike ros2_so_arm's MJCF site. -->
                   <site group="5" name="end_effector_link" pos="-0.0079 -0.000218121 -0.0981274" quat="0.707105 0 0.707108 0"/>
-                  <!-- Recomputed from our own gripper_xyz/gripper_rpy (no pitch offset), unlike
-                       ros2_so_arm's so_arm101_macro.xacro (undocumented 0.18 rad offset). -->
+                  <!-- Recomputed from our own gripper_rpy (no pitch offset), unlike ros2_so_arm's macro. -->
                   <body name="moving_jaw_link" pos="0.0202 0.0188 -0.0234" quat="0.707105 0.707108 0 0">
                     <joint axis="0 0 1" name="gripper_joint" range="-0.174533 1.74533" class="sts3215"/>
@@ -248,7 +266,9 @@
         <exclude body1="wrist_link" body2="gripper_link"/>
         <exclude body1="gripper_link" body2="moving_jaw_link"/>
-        <exclude body1="gripper_link" body2="wrist_camera_mount_link"/>
-        <exclude body1="wrist_camera_mount_link" body2="wrist_camera_body_link"/>
-        <exclude body1="gripper_link" body2="wrist_camera_body_link"/>
+        <xacro:if value="${'$(arg wrist_camera_mjcf)' == 'true'}">
+          <exclude body1="gripper_link" body2="wrist_camera_mount_link"/>
+          <exclude body1="wrist_camera_mount_link" body2="wrist_camera_body_link"/>
+          <exclude body1="gripper_link" body2="wrist_camera_body_link"/>
+        </xacro:if>
       </contact>
       <worldbody>
@@ -257,6 +277,5 @@
     </xacro:if>
   </xacro:if>
-  <!-- Compares $(arg standalone) directly, not via a bridged property - xacro auto-coerces
-       "true"/"false" properties to Python bool, breaking a naive string comparison. -->
+  <!-- Compares $(arg standalone) directly - xacro auto-coerces bridged properties to Python bool. -->
   <xacro:if value="${'$(arg standalone)' == 'true'}">
     <statistic center="0.1 -0.01 0.05" extent="0.5"/>
