Commit message: Restore per-joint PID coefficients and add commented internal_* EEPROM tuning template

File: so_arm_description/urdf/so100/so100.control.xacro (robot description, xacro)
@@ -23,7 +23,22 @@
   <xacro:property name="max_torque_nm" value="2.942"/>  <!-- N⋅m (30 kgf⋅cm for STS3215) -->
   <!-- Position-mode (Mode 0) internal servo PID, written to EEPROM on activate -->
-  <xacro:property name="p_coefficient" value="14"/>
-  <xacro:property name="d_coefficient" value="24"/>
-  <xacro:property name="i_coefficient" value="0"/>
+  <xacro:property name="shoulder_pan_p_coefficient" value="14"/>
+  <xacro:property name="shoulder_pan_d_coefficient" value="24"/>
+  <xacro:property name="shoulder_pan_i_coefficient" value="0"/>
+  <xacro:property name="shoulder_lift_p_coefficient" value="14"/>
+  <xacro:property name="shoulder_lift_d_coefficient" value="24"/>
+  <xacro:property name="shoulder_lift_i_coefficient" value="0"/>
+  <xacro:property name="elbow_flex_p_coefficient" value="14"/>
+  <xacro:property name="elbow_flex_d_coefficient" value="24"/>
+  <xacro:property name="elbow_flex_i_coefficient" value="0"/>
+  <xacro:property name="wrist_flex_p_coefficient" value="14"/>
+  <xacro:property name="wrist_flex_d_coefficient" value="24"/>
+  <xacro:property name="wrist_flex_i_coefficient" value="0"/>
+  <xacro:property name="wrist_roll_p_coefficient" value="14"/>
+  <xacro:property name="wrist_roll_d_coefficient" value="24"/>
+  <xacro:property name="wrist_roll_i_coefficient" value="0"/>
+  <xacro:property name="gripper_p_coefficient" value="14"/>
+  <xacro:property name="gripper_d_coefficient" value="24"/>
+  <xacro:property name="gripper_i_coefficient" value="0"/>
   <!-- Position insensitive-area (CW_DEAD/CCW_DEAD, both set to this value) -->
   <xacro:property name="deadband" value="10"/>

File: so_arm_description/urdf/so100/so100.urdf.xacro (robot description, xacro)
@@ -16,7 +16,22 @@
   <xacro:arg name="wrist_roll_motor_id" default="${wrist_roll_motor_id}"/>
   <xacro:arg name="gripper_motor_id" default="${gripper_motor_id}"/>
-  <xacro:arg name="p_coefficient" default="${p_coefficient}"/>
-  <xacro:arg name="d_coefficient" default="${d_coefficient}"/>
-  <xacro:arg name="i_coefficient" default="${i_coefficient}"/>
+  <xacro:arg name="shoulder_pan_p_coefficient" default="${shoulder_pan_p_coefficient}"/>
+  <xacro:arg name="shoulder_pan_d_coefficient" default="${shoulder_pan_d_coefficient}"/>
+  <xacro:arg name="shoulder_pan_i_coefficient" default="${shoulder_pan_i_coefficient}"/>
+  <xacro:arg name="shoulder_lift_p_coefficient" default="${shoulder_lift_p_coefficient}"/>
+  <xacro:arg name="shoulder_lift_d_coefficient" default="${shoulder_lift_d_coefficient}"/>
+  <xacro:arg name="shoulder_lift_i_coefficient" default="${shoulder_lift_i_coefficient}"/>
+  <xacro:arg name="elbow_flex_p_coefficient" default="${elbow_flex_p_coefficient}"/>
+  <xacro:arg name="elbow_flex_d_coefficient" default="${elbow_flex_d_coefficient}"/>
+  <xacro:arg name="elbow_flex_i_coefficient" default="${elbow_flex_i_coefficient}"/>
+  <xacro:arg name="wrist_flex_p_coefficient" default="${wrist_flex_p_coefficient}"/>
+  <xacro:arg name="wrist_flex_d_coefficient" default="${wrist_flex_d_coefficient}"/>
+  <xacro:arg name="wrist_flex_i_coefficient" default="${wrist_flex_i_coefficient}"/>
+  <xacro:arg name="wrist_roll_p_coefficient" default="${wrist_roll_p_coefficient}"/>
+  <xacro:arg name="wrist_roll_d_coefficient" default="${wrist_roll_d_coefficient}"/>
+  <xacro:arg name="wrist_roll_i_coefficient" default="${wrist_roll_i_coefficient}"/>
+  <xacro:arg name="gripper_p_coefficient" default="${gripper_p_coefficient}"/>
+  <xacro:arg name="gripper_d_coefficient" default="${gripper_d_coefficient}"/>
+  <xacro:arg name="gripper_i_coefficient" default="${gripper_i_coefficient}"/>
   <xacro:arg name="deadband" default="${deadband}"/>
   <!-- real=STS serial plugin, mujoco=MujocoSystemInterface, mock_components=GenericSystem. -->
@@ -350,8 +365,15 @@
       <param name="max_velocity">${max_velocity_rads}</param>
       <param name="position_center_steps">2048</param>
-      <param name="p_coefficient">$(arg p_coefficient)</param>
-      <param name="d_coefficient">$(arg d_coefficient)</param>
-      <param name="i_coefficient">$(arg i_coefficient)</param>
+      <param name="p_coefficient">$(arg shoulder_pan_p_coefficient)</param>
+      <param name="d_coefficient">$(arg shoulder_pan_d_coefficient)</param>
+      <param name="i_coefficient">$(arg shoulder_pan_i_coefficient)</param>
       <param name="deadband">$(arg deadband)</param>
+      <!-- Undocumented STS3215 EEPROM tuning registers (community-discovered). Uncomment to enable;
+           internal_max_vel/internal_max_acc/internal_acc_coeff: [0,254], internal_control_period: [1,254].
+      <param name="internal_max_vel">65</param>
+      <param name="internal_max_acc">254</param>
+      <param name="internal_acc_coeff">0</param>
+      <param name="internal_control_period">20</param>
+      -->
       <!-- cmd interfaces depend on arm_operating_mode -->
       <xacro:if value="${'$(arg arm_operating_mode)' == '2'}">
@@ -382,8 +404,15 @@
       <param name="max_velocity">${max_velocity_rads}</param>
       <param name="position_center_steps">2048</param>
-      <param name="p_coefficient">$(arg p_coefficient)</param>
-      <param name="d_coefficient">$(arg d_coefficient)</param>
-      <param name="i_coefficient">$(arg i_coefficient)</param>
+      <param name="p_coefficient">$(arg shoulder_lift_p_coefficient)</param>
+      <param name="d_coefficient">$(arg shoulder_lift_d_coefficient)</param>
+      <param name="i_coefficient">$(arg shoulder_lift_i_coefficient)</param>
       <param name="deadband">$(arg deadband)</param>
+      <!-- Undocumented STS3215 EEPROM tuning registers (community-discovered). Uncomment to enable;
+           internal_max_vel/internal_max_acc/internal_acc_coeff: [0,254], internal_control_period: [1,254].
+      <param name="internal_max_vel">65</param>
+      <param name="internal_max_acc">254</param>
+      <param name="internal_acc_coeff">0</param>
+      <param name="internal_control_period">20</param>
+      -->
       <!-- cmd interfaces depend on arm_operating_mode -->
       <xacro:if value="${'$(arg arm_operating_mode)' == '2'}">
@@ -414,8 +443,15 @@
       <param name="max_velocity">${max_velocity_rads}</param>
       <param name="position_center_steps">2048</param>
-      <param name="p_coefficient">$(arg p_coefficient)</param>
-      <param name="d_coefficient">$(arg d_coefficient)</param>
-      <param name="i_coefficient">$(arg i_coefficient)</param>
+      <param name="p_coefficient">$(arg elbow_flex_p_coefficient)</param>
+      <param name="d_coefficient">$(arg elbow_flex_d_coefficient)</param>
+      <param name="i_coefficient">$(arg elbow_flex_i_coefficient)</param>
       <param name="deadband">$(arg deadband)</param>
+      <!-- Undocumented STS3215 EEPROM tuning registers (community-discovered). Uncomment to enable;
+           internal_max_vel/internal_max_acc/internal_acc_coeff: [0,254], internal_control_period: [1,254].
+      <param name="internal_max_vel">65</param>
+      <param name="internal_max_acc">254</param>
+      <param name="internal_acc_coeff">0</param>
+      <param name="internal_control_period">20</param>
+      -->
       <!-- cmd interfaces depend on arm_operating_mode -->
       <xacro:if value="${'$(arg arm_operating_mode)' == '2'}">
@@ -446,8 +482,15 @@
       <param name="max_velocity">${max_velocity_rads}</param>
       <param name="position_center_steps">2048</param>
-      <param name="p_coefficient">$(arg p_coefficient)</param>
-      <param name="d_coefficient">$(arg d_coefficient)</param>
-      <param name="i_coefficient">$(arg i_coefficient)</param>
+      <param name="p_coefficient">$(arg wrist_flex_p_coefficient)</param>
+      <param name="d_coefficient">$(arg wrist_flex_d_coefficient)</param>
+      <param name="i_coefficient">$(arg wrist_flex_i_coefficient)</param>
       <param name="deadband">$(arg deadband)</param>
+      <!-- Undocumented STS3215 EEPROM tuning registers (community-discovered). Uncomment to enable;
+           internal_max_vel/internal_max_acc/internal_acc_coeff: [0,254], internal_control_period: [1,254].
+      <param name="internal_max_vel">65</param>
+      <param name="internal_max_acc">254</param>
+      <param name="internal_acc_coeff">0</param>
+      <param name="internal_control_period">20</param>
+      -->
       <!-- cmd interfaces depend on arm_operating_mode -->
       <xacro:if value="${'$(arg arm_operating_mode)' == '2'}">
@@ -478,8 +521,15 @@
       <param name="max_velocity">${max_velocity_rads}</param>
       <param name="position_center_steps">2048</param>
-      <param name="p_coefficient">$(arg p_coefficient)</param>
-      <param name="d_coefficient">$(arg d_coefficient)</param>
-      <param name="i_coefficient">$(arg i_coefficient)</param>
+      <param name="p_coefficient">$(arg wrist_roll_p_coefficient)</param>
+      <param name="d_coefficient">$(arg wrist_roll_d_coefficient)</param>
+      <param name="i_coefficient">$(arg wrist_roll_i_coefficient)</param>
       <param name="deadband">$(arg deadband)</param>
+      <!-- Undocumented STS3215 EEPROM tuning registers (community-discovered). Uncomment to enable;
+           internal_max_vel/internal_max_acc/internal_acc_coeff: [0,254], internal_control_period: [1,254].
+      <param name="internal_max_vel">65</param>
+      <param name="internal_max_acc">254</param>
+      <param name="internal_acc_coeff">0</param>
+      <param name="internal_control_period">20</param>
+      -->
       <!-- cmd interfaces depend on arm_operating_mode -->
       <xacro:if value="${'$(arg arm_operating_mode)' == '2'}">
@@ -510,8 +560,15 @@
       <param name="max_velocity">${max_velocity_rads}</param>
       <param name="position_center_steps">2048</param>
-      <param name="p_coefficient">$(arg p_coefficient)</param>
-      <param name="d_coefficient">$(arg d_coefficient)</param>
-      <param name="i_coefficient">$(arg i_coefficient)</param>
+      <param name="p_coefficient">$(arg gripper_p_coefficient)</param>
+      <param name="d_coefficient">$(arg gripper_d_coefficient)</param>
+      <param name="i_coefficient">$(arg gripper_i_coefficient)</param>
       <param name="deadband">$(arg deadband)</param>
+      <!-- Undocumented STS3215 EEPROM tuning registers (community-discovered). Uncomment to enable;
+           internal_max_vel/internal_max_acc/internal_acc_coeff: [0,254], internal_control_period: [1,254].
+      <param name="internal_max_vel">65</param>
+      <param name="internal_max_acc">254</param>
+      <param name="internal_acc_coeff">0</param>
+      <param name="internal_control_period">20</param>
+      -->
       <!-- cmd interfaces depend on gripper_operating_mode -->
       <xacro:if value="${'$(arg gripper_operating_mode)' == '2'}">

File: so_arm_description/urdf/so101/so101.control.xacro (robot description, xacro)
@@ -23,7 +23,22 @@
   <xacro:property name="max_torque_nm" value="2.942"/>  <!-- N⋅m (30 kgf⋅cm for STS3215) -->
   <!-- Position-mode (Mode 0) internal servo PID, written to EEPROM on activate -->
-  <xacro:property name="p_coefficient" value="14"/>
-  <xacro:property name="d_coefficient" value="24"/>
-  <xacro:property name="i_coefficient" value="0"/>
+  <xacro:property name="shoulder_pan_p_coefficient" value="14"/>
+  <xacro:property name="shoulder_pan_d_coefficient" value="24"/>
+  <xacro:property name="shoulder_pan_i_coefficient" value="0"/>
+  <xacro:property name="shoulder_lift_p_coefficient" value="14"/>
+  <xacro:property name="shoulder_lift_d_coefficient" value="24"/>
+  <xacro:property name="shoulder_lift_i_coefficient" value="0"/>
+  <xacro:property name="elbow_flex_p_coefficient" value="14"/>
+  <xacro:property name="elbow_flex_d_coefficient" value="24"/>
+  <xacro:property name="elbow_flex_i_coefficient" value="0"/>
+  <xacro:property name="wrist_flex_p_coefficient" value="14"/>
+  <xacro:property name="wrist_flex_d_coefficient" value="24"/>
+  <xacro:property name="wrist_flex_i_coefficient" value="0"/>
+  <xacro:property name="wrist_roll_p_coefficient" value="14"/>
+  <xacro:property name="wrist_roll_d_coefficient" value="24"/>
+  <xacro:property name="wrist_roll_i_coefficient" value="0"/>
+  <xacro:property name="gripper_p_coefficient" value="14"/>
+  <xacro:property name="gripper_d_coefficient" value="24"/>
+  <xacro:property name="gripper_i_coefficient" value="0"/>
   <!-- Position insensitive-area (CW_DEAD/CCW_DEAD, both set to this value) -->
   <xacro:property name="deadband" value="10"/>

File: so_arm_description/urdf/so101/so101.urdf.xacro (robot description, xacro)
@@ -16,7 +16,22 @@
   <xacro:arg name="wrist_roll_motor_id" default="${wrist_roll_motor_id}"/>
   <xacro:arg name="gripper_motor_id" default="${gripper_motor_id}"/>
-  <xacro:arg name="p_coefficient" default="${p_coefficient}"/>
-  <xacro:arg name="d_coefficient" default="${d_coefficient}"/>
-  <xacro:arg name="i_coefficient" default="${i_coefficient}"/>
+  <xacro:arg name="shoulder_pan_p_coefficient" default="${shoulder_pan_p_coefficient}"/>
+  <xacro:arg name="shoulder_pan_d_coefficient" default="${shoulder_pan_d_coefficient}"/>
+  <xacro:arg name="shoulder_pan_i_coefficient" default="${shoulder_pan_i_coefficient}"/>
+  <xacro:arg name="shoulder_lift_p_coefficient" default="${shoulder_lift_p_coefficient}"/>
+  <xacro:arg name="shoulder_lift_d_coefficient" default="${shoulder_lift_d_coefficient}"/>
+  <xacro:arg name="shoulder_lift_i_coefficient" default="${shoulder_lift_i_coefficient}"/>
+  <xacro:arg name="elbow_flex_p_coefficient" default="${elbow_flex_p_coefficient}"/>
+  <xacro:arg name="elbow_flex_d_coefficient" default="${elbow_flex_d_coefficient}"/>
+  <xacro:arg name="elbow_flex_i_coefficient" default="${elbow_flex_i_coefficient}"/>
+  <xacro:arg name="wrist_flex_p_coefficient" default="${wrist_flex_p_coefficient}"/>
+  <xacro:arg name="wrist_flex_d_coefficient" default="${wrist_flex_d_coefficient}"/>
+  <xacro:arg name="wrist_flex_i_coefficient" default="${wrist_flex_i_coefficient}"/>
+  <xacro:arg name="wrist_roll_p_coefficient" default="${wrist_roll_p_coefficient}"/>
+  <xacro:arg name="wrist_roll_d_coefficient" default="${wrist_roll_d_coefficient}"/>
+  <xacro:arg name="wrist_roll_i_coefficient" default="${wrist_roll_i_coefficient}"/>
+  <xacro:arg name="gripper_p_coefficient" default="${gripper_p_coefficient}"/>
+  <xacro:arg name="gripper_d_coefficient" default="${gripper_d_coefficient}"/>
+  <xacro:arg name="gripper_i_coefficient" default="${gripper_i_coefficient}"/>
   <xacro:arg name="deadband" default="${deadband}"/>
   <!-- real=STS serial plugin, mujoco=MujocoSystemInterface, mock_components=GenericSystem. -->
@@ -487,8 +502,15 @@
       <param name="max_velocity">${max_velocity_rads}</param>
       <param name="position_center_steps">2048</param>
-      <param name="p_coefficient">$(arg p_coefficient)</param>
-      <param name="d_coefficient">$(arg d_coefficient)</param>
-      <param name="i_coefficient">$(arg i_coefficient)</param>
+      <param name="p_coefficient">$(arg shoulder_pan_p_coefficient)</param>
+      <param name="d_coefficient">$(arg shoulder_pan_d_coefficient)</param>
+      <param name="i_coefficient">$(arg shoulder_pan_i_coefficient)</param>
       <param name="deadband">$(arg deadband)</param>
+      <!-- Undocumented STS3215 EEPROM tuning registers (community-discovered). Uncomment to enable;
+           internal_max_vel/internal_max_acc/internal_acc_coeff: [0,254], internal_control_period: [1,254].
+      <param name="internal_max_vel">65</param>
+      <param name="internal_max_acc">254</param>
+      <param name="internal_acc_coeff">0</param>
+      <param name="internal_control_period">20</param>
+      -->
       <!-- cmd interfaces depend on arm_operating_mode -->
       <xacro:if value="${'$(arg arm_operating_mode)' == '2'}">
@@ -519,8 +541,15 @@
       <param name="max_velocity">${max_velocity_rads}</param>
       <param name="position_center_steps">2048</param>
-      <param name="p_coefficient">$(arg p_coefficient)</param>
-      <param name="d_coefficient">$(arg d_coefficient)</param>
-      <param name="i_coefficient">$(arg i_coefficient)</param>
+      <param name="p_coefficient">$(arg shoulder_lift_p_coefficient)</param>
+      <param name="d_coefficient">$(arg shoulder_lift_d_coefficient)</param>
+      <param name="i_coefficient">$(arg shoulder_lift_i_coefficient)</param>
       <param name="deadband">$(arg deadband)</param>
+      <!-- Undocumented STS3215 EEPROM tuning registers (community-discovered). Uncomment to enable;
+           internal_max_vel/internal_max_acc/internal_acc_coeff: [0,254], internal_control_period: [1,254].
+      <param name="internal_max_vel">65</param>
+      <param name="internal_max_acc">254</param>
+      <param name="internal_acc_coeff">0</param>
+      <param name="internal_control_period">20</param>
+      -->
       <!-- cmd interfaces depend on arm_operating_mode -->
       <xacro:if value="${'$(arg arm_operating_mode)' == '2'}">
@@ -551,8 +580,15 @@
       <param name="max_velocity">${max_velocity_rads}</param>
       <param name="position_center_steps">2048</param>
-      <param name="p_coefficient">$(arg p_coefficient)</param>
-      <param name="d_coefficient">$(arg d_coefficient)</param>
-      <param name="i_coefficient">$(arg i_coefficient)</param>
+      <param name="p_coefficient">$(arg elbow_flex_p_coefficient)</param>
+      <param name="d_coefficient">$(arg elbow_flex_d_coefficient)</param>
+      <param name="i_coefficient">$(arg elbow_flex_i_coefficient)</param>
       <param name="deadband">$(arg deadband)</param>
+      <!-- Undocumented STS3215 EEPROM tuning registers (community-discovered). Uncomment to enable;
+           internal_max_vel/internal_max_acc/internal_acc_coeff: [0,254], internal_control_period: [1,254].
+      <param name="internal_max_vel">65</param>
+      <param name="internal_max_acc">254</param>
+      <param name="internal_acc_coeff">0</param>
+      <param name="internal_control_period">20</param>
+      -->
       <!-- cmd interfaces depend on arm_operating_mode -->
       <xacro:if value="${'$(arg arm_operating_mode)' == '2'}">
@@ -583,8 +619,15 @@
       <param name="max_velocity">${max_velocity_rads}</param>
       <param name="position_center_steps">2048</param>
-      <param name="p_coefficient">$(arg p_coefficient)</param>
-      <param name="d_coefficient">$(arg d_coefficient)</param>
-      <param name="i_coefficient">$(arg i_coefficient)</param>
+      <param name="p_coefficient">$(arg wrist_flex_p_coefficient)</param>
+      <param name="d_coefficient">$(arg wrist_flex_d_coefficient)</param>
+      <param name="i_coefficient">$(arg wrist_flex_i_coefficient)</param>
       <param name="deadband">$(arg deadband)</param>
+      <!-- Undocumented STS3215 EEPROM tuning registers (community-discovered). Uncomment to enable;
+           internal_max_vel/internal_max_acc/internal_acc_coeff: [0,254], internal_control_period: [1,254].
+      <param name="internal_max_vel">65</param>
+      <param name="internal_max_acc">254</param>
+      <param name="internal_acc_coeff">0</param>
+      <param name="internal_control_period">20</param>
+      -->
       <!-- cmd interfaces depend on arm_operating_mode -->
       <xacro:if value="${'$(arg arm_operating_mode)' == '2'}">
@@ -615,8 +658,15 @@
       <param name="max_velocity">${max_velocity_rads}</param>
       <param name="position_center_steps">2048</param>
-      <param name="p_coefficient">$(arg p_coefficient)</param>
-      <param name="d_coefficient">$(arg d_coefficient)</param>
-      <param name="i_coefficient">$(arg i_coefficient)</param>
+      <param name="p_coefficient">$(arg wrist_roll_p_coefficient)</param>
+      <param name="d_coefficient">$(arg wrist_roll_d_coefficient)</param>
+      <param name="i_coefficient">$(arg wrist_roll_i_coefficient)</param>
       <param name="deadband">$(arg deadband)</param>
+      <!-- Undocumented STS3215 EEPROM tuning registers (community-discovered). Uncomment to enable;
+           internal_max_vel/internal_max_acc/internal_acc_coeff: [0,254], internal_control_period: [1,254].
+      <param name="internal_max_vel">65</param>
+      <param name="internal_max_acc">254</param>
+      <param name="internal_acc_coeff">0</param>
+      <param name="internal_control_period">20</param>
+      -->
       <!-- cmd interfaces depend on arm_operating_mode -->
       <xacro:if value="${'$(arg arm_operating_mode)' == '2'}">
@@ -647,8 +697,15 @@
       <param name="max_velocity">${max_velocity_rads}</param>
       <param name="position_center_steps">2048</param>
-      <param name="p_coefficient">$(arg p_coefficient)</param>
-      <param name="d_coefficient">$(arg d_coefficient)</param>
-      <param name="i_coefficient">$(arg i_coefficient)</param>
+      <param name="p_coefficient">$(arg gripper_p_coefficient)</param>
+      <param name="d_coefficient">$(arg gripper_d_coefficient)</param>
+      <param name="i_coefficient">$(arg gripper_i_coefficient)</param>
       <param name="deadband">$(arg deadband)</param>
+      <!-- Undocumented STS3215 EEPROM tuning registers (community-discovered). Uncomment to enable;
+           internal_max_vel/internal_max_acc/internal_acc_coeff: [0,254], internal_control_period: [1,254].
+      <param name="internal_max_vel">65</param>
+      <param name="internal_max_acc">254</param>
+      <param name="internal_acc_coeff">0</param>
+      <param name="internal_control_period">20</param>
+      -->
       <!-- cmd interfaces depend on gripper_operating_mode -->
       <xacro:if value="${'$(arg gripper_operating_mode)' == '2'}">
